File: projects/ESP_DEV_BOARD/ESP_DEV_BOARD.kicad_pcb (KiCad board)
At the start: 2 copper layers, 76 x 92 mm, 38 parts, among them CN1 MJ-179P, CN2 B6B-XH-A, CN3 DM3AT-SF-PEJM5, CN7 PH-1X10RG(2), SW1 SKHHBY, SW2 SKHHBY, SW3 SKHHBY, SW4 SKHHBY, U1 BME680, U2 CCS811

Commit message: 赤外線送受信回路の追加。
Parts:
- added C5: 47uF/16V, A01myFootPrint:CP_Radial_D5.0mm_P2.00mm, F.Cu at (57.0, 72.9)
- added IC1: OSRB38C9AA, A01myFootPrint:ic_OSRB38C9AA, F.Cu at (54.4, 69.1)
- added JP1: JUMPER2*1, A01myFootPrint:JP_JUMPER1x2, F.Cu at (55.7, 79.9)
- added JP2: JUMPER2*1, A01myFootPrint:JP_JUMPER1x2, F.Cu at (55.7, 77.3)
- added LED3: Ir LED, A01myFootPrint:led_5mmLED, F.Cu at (53.8, 84.9)
- added R13: 100, A01myFootPrint:C_0603, B.Cu at (60.8, 69.1)
- added R14: 20K, A01myFootPrint:C_0603, B.Cu at (60.8, 76.7)
- added R15: 47, A01myFootPrint:C_0603, B.Cu at (57.6, 83.7)
- moved TP2 66.0 mm to (79.2, 122.4)
- moved CN2 1.91 mm to (53.8, 97.6)
Routing:
- net /RXD1: track 66.8 -> 93.2 mm
- net /1PPS: track 65.4 -> 88.3 mm
- net Net-(IC1-Pad1): track 0.00 -> 9.31 mm
- net Net-(C5-Pad1): track 0.00 -> 6.82 mm
- net +3V3: track 210.0 -> 216.0 mm, vias 11 -> 13
- net GND: track 498.6 -> 493.1 mm, vias 17 -> 18
- net Net-(JP1-Pad2): track 0.00 -> 3.27 mm
- net Net-(LED3-Pad1): track 0.00 -> 2.73 mm
- net +5V: track 107.8 -> 108.6 mm
- net /TXD1: track 50.3 -> 49.5 mm
