File: projects/2110/2110_LOW_THRESHOLD_SHORT_CHECKER.sch (KiCad schematic (older format))
At the start: 25 parts, among them CN2 2PIN, IC1 AD823AN, IC11 AD823AN, SW1 SS12D01G4

Commit message: R2の追加。
Parts:
- added R2: 1K, symbol register:R
Connections:
- net at IC1.1, R1.1, R6.1: now also R2.2; no longer C4.1
- new net: C4.1, R2.1
Other:
- moved on the sheet: BZ1, C4, D5, D6
Changed lines of the file:
@@
 L diode:DIODE D5
 U 1 1 61236DBF
-P 7300 2750
-F 0 "D5" V 7300 2650 50  0000 R CNN
-F 1 "1S2076A" V 7200 2650 50  0000 R CNN
-F 2 "" H 7300 2750 60  0001 C CNN
-F 3 "" H 7300 2750 60  0001 C CNN
-	1    7300 2750
+P 7650 2750
+F 0 "D5" V 7650 2650 50  0000 R CNN
+F 1 "1S2076A" V 7550 2650 50  0000 R CNN
+F 2 "" H 7650 2750 60  0001 C CNN
+F 3 "" H 7650 2750 60  0001 C CNN
+	1    7650 2750
 	0    -1   -1   0
 $EndComp
@@
 L diode:DIODE D6
 U 1 1 61237C9B
-P 7300 3150
-F 0 "D6" V 7300 3050 50  0000 R CNN
-F 1 "1S2076A" V 7200 3050 50  0000 R CNN
-F 2 "" H 7300 3150 60  0001 C CNN
-F 3 "" H 7300 3150 60  0001 C CNN
-	1    7300 3150
+P 7650 3150
+F 0 "D6" V 7650 3050 50  0000 R CNN
+F 1 "1S2076A" V 7550 3050 50  0000 R CNN
+F 2 "" H 7650 3150 60  0001 C CNN
+F 3 "" H 7650 3150 60  0001 C CNN
+	1    7650 3150
 	0    -1   -1   0
 $EndComp
@@
 L capacitor:CP1_Small C4
 U 1 1 6123AE03
-P 7050 2950
-F 0 "C4" V 7278 2950 50  0000 C CNN
-F 1 "220uF/16V" V 7187 2950 50  0000 C CNN
-F 2 "" H 7050 2950 50  0001 C CNN
-F 3 "" H 7050 2950 50  0001 C CNN
-	1    7050 2950
+P 7400 2950
+F 0 "C4" V 7628 2950 50  0000 C CNN
+F 1 "220uF/16V" V 7537 2950 50  0000 C CNN
+F 2 "" H 7400 2950 50  0001 C CNN
+F 3 "" H 7400 2950 50  0001 C CNN
+	1    7400 2950
 	0    -1   -1   0
 $EndComp
@@
 L SPEAKER:BUZZER BZ1
 U 1 1 61245DB8
-P 7850 3150
-F 0 "BZ1" V 7804 3238 50  0000 L CNN
-F 1 "PKM13EPYH4000-A0" V 7895 3238 50  0000 L CNN
-F 2 "" H 7850 3150 50  0001 C CNN
-F 3 "" H 7850 3150 50  0001 C CNN
-	1    7850 3150
+P 8200 3150
+F 0 "BZ1" V 8154 3238 50  0000 L CNN
+F 1 "PKM13EPYH4000-A0" V 8245 3238 50  0000 L CNN
+F 2 "" H 8200 3150 50  0001 C CNN
+F 3 "" H 8200 3150 50  0001 C CNN
+	1    8200 3150
 	0    1    1    0
 $EndComp
@@
 L power:GND #PWR0117
 U 1 1 6124704B
-P 7850 3350
-F 0 "#PWR0117" H 7850 3100 50  0001 C CNN
-F 1 "GND" H 7855 3177 50  0000 C CNN
-F 2 "" H 7850 3350 50  0001 C CNN
-F 3 "" H 7850 3350 50  0001 C CNN
-	1    7850 3350
+P 8200 3350
+F 0 "#PWR0117" H 8200 3100 50  0001 C CNN
+F 1 "GND" H 8205 3177 50  0000 C CNN
+F 2 "" H 8200 3350 50  0001 C CNN
+F 3 "" H 8200 3350 50  0001 C CNN
+	1    8200 3350
 	1    0    0    -1
 $EndComp
@@
 L power:+9V #PWR0118
 U 1 1 6124958A
-P 7300 2550
-F 0 "#PWR0118" H 7300 2400 50  0001 C CNN
-F 1 "+9V" H 7315 2723 50  0000 C CNN
-F 2 "" H 7300 2550 50  0001 C CNN
-F 3 "" H 7300 2550 50  0001 C CNN
-	1    7300 2550
+P 7650 2550
+F 0 "#PWR0118" H 7650 2400 50  0001 C CNN
+F 1 "+9V" H 7665 2723 50  0000 C CNN
+F 2 "" H 7650 2550 50  0001 C CNN
+F 3 "" H 7650 2550 50  0001 C CNN
+	1    7650 2550
 	1    0    0    -1
 $EndComp
 Wire Wire Line
-	7300 2550 7300 2600
+	7650 2550 7650 2600
 Wire Wire Line
-	7300 2900 7300 2950
+	7650 2900 7650 2950
 Wire Wire Line
-	7150 2950 7300 2950
-Connection ~ 7300 2950
+	7500 2950 7650 2950
+Connection ~ 7650 2950
 Wire Wire Line
-	7300 2950 7300 3000
+	7650 2950 7650 3000
 Wire Wire Line
-	6950 2950 6800 2950
+	6900 2950 6800 2950
 $Comp
 L power:GND #PWR0119
 U 1 1 6125029B
-P 7300 3350
-F 0 "#PWR0119" H 7300 3100 50  0001 C CNN
-F 1 "GND" H 7305 3177 50  0000 C CNN
-F 2 "" H 7300 3350 50  0001 C CNN
-F 3 "" H 7300 3350 50  0001 C CNN
-	1    7300 3350
+P 7650 3350
+F 0 "#PWR0119" H 7650 3100 50  0001 C CNN
+F 1 "GND" H 7655 3177 50  0000 C CNN
+F 2 "" H 7650 3350 50  0001 C CNN
+F 3 "" H 7650 3350 50  0001 C CNN
+	1    7650 3350
 	1    0    0    -1
 $EndComp
 Wire Wire Line
-	7300 3350 7300 3300
+	7650 3350 7650 3300
 Wire Wire Line
-	7850 3000 7850 2950
+	8200 3000 8200 2950
 Wire Wire Line
-	7850 2950 7300 2950
+	8200 2950 7650 2950
 Wire Wire Line
-	7850 3300 7850 3350
+	8200 3300 8200 3350
 Text Notes 3250 1150 0    50   ~ 0
 006P BATTERY HOLDER
@@
 Text Notes 5900 2000 0    50   ~ 0
 0.7V
+$Comp
+L register:R R2
+U 1 1 611E510C
+P 7050 2950
+F 0 "R2" V 6950 2900 50  0000 L CNN
+F 1 "1K" V 7050 2900 50  0000 L CNN
+F 2 "" V 6980 2950 50  0001 C CNN
+F 3 "" H 7050 2950 50  0001 C CNN
+	1    7050 2950
+	0    1    1    0
+$EndComp
+Wire Wire Line
+	7300 2950 7200 2950
 $EndSCHEMATC
